File: password_manager.kicad_pcb (KiCad board)
At the start: 2 copper layers, 100 x 100 mm, 12 parts, among them J1 Micro_SD_Card_Det2, J2 Micro_SD_Card_Det2, J3 Micro_SD_Card_Det2, U1 STM32H743VITx, X1 25MHz

Commit message: nowe libs
Parts:
- added J4: USB_C_Receptacle_USB2.0, Connector_USB:USB_C_Receptacle_GCT_USB4105-xx-A_16P_TopMnt_Horizontal, F.Cu at (58.8, 122.4)
- added J5: zasilanie, Connector_USB:USB_C_Receptacle_GCT_USB4105-xx-A_16P_TopMnt_Horizontal, F.Cu at (58.7, 133.6)
- added P1: PS/2, password_manager_foots:Connector_Mini-DIN_Female_6Pin_2rows, F.Cu at (140.2, 100.8)
- added SW1_1: SW_1, Button_Switch_SMD:SW_Push_1P1T_NO_6x6mm_H9.5mm, F.Cu at (120.9, 140.7)
- added SW1_2: SW_2, Button_Switch_SMD:SW_Push_1P1T_NO_6x6mm_H9.5mm, F.Cu at (120.9, 133.1)
- added SW1_3: SW_3, Button_Switch_SMD:SW_Push_1P1T_NO_6x6mm_H9.5mm, F.Cu at (120.9, 125.5)
- added SW1_4: SW_4, Button_Switch_SMD:SW_Push_1P1T_NO_6x6mm_H9.5mm, F.Cu at (120.9, 117.9)
- added SW2_1: SW_1, Button_Switch_SMD:SW_Push_1P1T_NO_6x6mm_H9.5mm, F.Cu at (109.8, 140.7)
- added SW2_2: SW_1, Button_Switch_SMD:SW_Push_1P1T_NO_6x6mm_H9.5mm, F.Cu at (109.8, 133.1)
- added SW2_3: SW_1, Button_Switch_SMD:SW_Push_1P1T_NO_6x6mm_H9.5mm, F.Cu at (109.8, 125.5)
- added SW2_4: SW_1, Button_Switch_SMD:SW_Push_1P1T_NO_6x6mm_H9.5mm, F.Cu at (109.8, 117.9)
- added SW3_1: SW_1, Button_Switch_SMD:SW_Push_1P1T_NO_6x6mm_H9.5mm, F.Cu at (98.8, 140.7)
- added SW3_2: SW_1, Button_Switch_SMD:SW_Push_1P1T_NO_6x6mm_H9.5mm, F.Cu at (98.8, 133.1)
- added SW3_3: SW_1, Button_Switch_SMD:SW_Push_1P1T_NO_6x6mm_H9.5mm, F.Cu at (98.8, 125.5)
- added SW3_4: SW_1, Button_Switch_SMD:SW_Push_1P1T_NO_6x6mm_H9.5mm, F.Cu at (98.8, 117.9)
- added SW4_1: SW_1, Button_Switch_SMD:SW_Push_1P1T_NO_6x6mm_H9.5mm, F.Cu at (87.7, 140.7)
- added SW4_2: SW_1, Button_Switch_SMD:SW_Push_1P1T_NO_6x6mm_H9.5mm, F.Cu at (87.7, 133.1)
- added SW4_3: SW_1, Button_Switch_SMD:SW_Push_1P1T_NO_6x6mm_H9.5mm, F.Cu at (87.7, 125.5)
- added SW4_4: SW_1, Button_Switch_SMD:SW_Push_1P1T_NO_6x6mm_H9.5mm, F.Cu at (87.7, 117.9)
- moved U1 12.5 mm to (95.0, 94.5)
- moved C1 7.11 mm to (110.3, 86.9)
- moved C2 7.11 mm to (110.3, 89.4)
- moved X1 7.11 mm to (114.2, 98.3)

Commit message: kolejne elementy
Parts:
- added CON1: ISP-10, foots:IDC-10_angled, B.Cu at (128.0, 64.8)
- added D1: LED_Small, Diode_SMD:D_0805_2012Metric_Pad1.15x1.40mm_HandSolder, F.Cu at (63.8, 60.2)
- added D2: LED_Small, Diode_SMD:D_0805_2012Metric_Pad1.15x1.40mm_HandSolder, F.Cu at (67.8, 60.5)
- added D3: LED_Small, Diode_SMD:D_0805_2012Metric_Pad1.15x1.40mm_HandSolder, F.Cu at (70.9, 60.5)
- added D4: LED_Small, Diode_SMD:D_0805_2012Metric_Pad1.15x1.40mm_HandSolder, F.Cu at (73.9, 60.5)
- added J10: Conn_01x22_Pin, Connector_PinHeader_2.54mm:PinHeader_1x22_P2.54mm_Vertical, F.Cu at (162.1, 156.4)
- added J11: masa_pomiarowa, foots:masa_pomiarowa, B.Cu at (55.1, 62.0)
- added J12: masa_pomiarowa, foots:masa_pomiarowa, B.Cu at (64.5, 144.3)
- added J13: masa_pomiarowa, foots:masa_pomiarowa, B.Cu at (145.5, 62.2)
- added J14: masa_pomiarowa, foots:masa_pomiarowa, B.Cu at (136.1, 145.0)
- added J15: LEDS, foots:4_PIN, F.Cu at (68.3, 54.9)
- added J16: test_pin, foots:3_PIN, F.Cu at (80.0, 54.2)
- added J17: test_pin, foots:3_PIN, F.Cu at (80.0, 57.9)
- added J18: test_pin, foots:3_PIN, F.Cu at (80.0, 61.6)
- added J19: test_pin, foots:3_PIN, F.Cu at (80.0, 65.3)
- added J20: test_pin, foots:3_PIN, F.Cu at (80.0, 69.0)
- added J21: test_pin, foots:3_PIN, F.Cu at (80.0, 72.6)
- added J6: RJ45_Shielded, password_manager_foots:RJ45_6339160-1_TE_Connectivity, F.Cu at (145.3, 79.2)
- added J7: Conn_01x22_Pin, Connector_PinHeader_2.54mm:PinHeader_1x22_P2.54mm_Horizontal, F.Cu at (162.1, 161.0)
- added J8: Conn_01x22_Pin, Connector_PinHeader_2.54mm:PinHeader_1x22_P2.54mm_Horizontal, F.Cu at (103.9, 162.1)
- added J9: Conn_01x22_Pin, Connector_PinHeader_2.54mm:PinHeader_1x22_P2.54mm_Vertical, F.Cu at (49.8, 153.9)
- added R1: R_Small, Resistor_SMD:R_0805_2012Metric_Pad1.20x1.40mm_HandSolder, F.Cu at (141.5, 126.3)
- added R2: 10K, Resistor_SMD:R_0805_2012Metric_Pad1.20x1.40mm_HandSolder, F.Cu at (141.5, 129.3)
- added SW1: SW_Push, Button_Switch_SMD:SW_Push_1P1T_NO_6x6mm_H9.5mm, F.Cu at (80.1, 84.4)
- moved J3 4.34 mm to (62.2, 104.4)
- moved J2 3.87 mm to (62.2, 88.4)
- moved U1 3.30 mm to (91.9, 95.8), turned to -45 degrees
- moved J1 3.08 mm to (62.2, 72.5)
- moved J4 1.52 mm to (58.9, 120.9)
- moved J5 0.54 mm to (58.9, 134.1)
Connections:
- U1 pad 14: unconnected-(U1-NRST-Pad14) -> Net-(U1-NRST)
