File: password_manager.kicad_sch (KiCad schematic)
At the start: 12 parts, among them J1 Micro_SD_Card_Det2, J2 Micro_SD_Card_Det2, J3 Micro_SD_Card_Det2, U1 STM32H743VITx, X1 25MHz

Commit message: nowe libs
Parts:
- added J4: USB_C_Receptacle_USB2.0, Connector_USB:USB_C_Receptacle_GCT_USB4105-xx-A_16P_TopMnt_Horizontal, symbol Connector:USB_C_Receptacle_USB2.0
- added J5: zasilanie, Connector_USB:USB_C_Receptacle_GCT_USB4105-xx-A_16P_TopMnt_Horizontal, symbol Connector:USB_C_Receptacle_USB2.0
- added P1: PS/2, password_manager_foots:Connector_Mini-DIN_Female_6Pin_2rows, symbol password_manager_symbols:Mini-DIN_6pins
Connections:
- net GND: now also J5.A1 (GND), J5.A12 (GND), J5.B1 (GND), J5.B12 (GND), J5.S1 (SHIELD)
- new net: J5.A4 (VBUS), J5.A9 (VBUS), J5.B4 (VBUS), J5.B9 (VBUS)
- new net: J4.A1 (GND), J4.A12 (GND), J4.B1 (GND), J4.B12 (GND)
- new net: J4.A4 (VBUS), J4.A9 (VBUS), J4.B4 (VBUS), J4.B9 (VBUS)
Changed lines of the file:
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@@
+    )
+  )
+  (symbol (lib_id "password_manager_symbols:Mini-DIN_6pins") (at 23.495 79.375 270) (mirror x) (unit 1)
+    (in_bom yes) (on_board yes) (dnp no)
+    (property "Reference" "P1" (at 17.145 80.645 90)
+      (effects (font (size 1.27 1.27)) (justify right))
+    )
+    (property "Value" "PS/2" (at 31.75 92.075 90)
+      (effects (font (size 1.27 1.27)) (justify right))
+    )
+    (property "Footprint" "password_manager_foots:Connector_Mini-DIN_Female_6Pin_2rows" (at 23.495 79.375 0)
+      (effects (font (size 1.27 1.27)) hide)
+    )
+    (property "Datasheet" "" (at 23.495 79.375 0)
+      (effects (font (size 1.27 1.27)))
+    )
+    (pin "1")
+    (pin "5")
+    (pin "4")
+    (pin "2")
+    (pin "3")
+    (pin "6")
+    (pin "7")
+    (instances
+      (project "password_manager"
+        (path "/c60f1c42-9579-4917-bb90-9d2f0e5f1bce"
+          (reference "P1") (unit 1)
+        )
+      )
     )
   )
@@
     )
   )
+  (symbol (lib_id "Connector:USB_C_Receptacle_USB2.0") (at 27.305 36.195 0) (unit 1)
+    (in_bom yes) (on_board yes) (dnp no)
+    (property "Reference" "J5" (at 27.305 13.97 0)
+      (effects (font (size 1.27 1.27)))
+    )
+    (property "Value" "zasilanie" (at 33.655 56.515 0)
+      (effects (font (size 1.27 1.27)))
+    )
+    (property "Footprint" "Connector_USB:USB_C_Receptacle_GCT_USB4105-xx-A_16P_TopMnt_Horizontal" (at 31.115 36.195 0)
+      (effects (font (size 1.27 1.27)) hide)
+    )
+    (property "Datasheet" "https://www.usb.org/sites/default/files/documents/usb_type-c.zip" (at 31.115 36.195 0)
+      (effects (font (size 1.27 1.27)) hide)
+    )
+    (pin "B4")
+    (pin "A5")
+    (pin "A1")
+    (pin "B6")
+    (pin "B8")
+    (pin "S1")
+    (pin "A12")
+    (pin "B7")
+    (pin "B1")
+    (pin "B5")
+    (pin "B12")
+    (pin "A7")
+    (pin "A4")
+    (pin "A9")
+    (pin "B9")
+    (pin "A6")
+    (pin "A8")
+    (instances
+      (project "password_manager"
+        (path "/c60f1c42-9579-4917-bb90-9d2f0e5f1bce"
+          (reference "J5") (unit 1)
+        )
+      )
+    )
+  )
   (symbol (lib_id "sp3jdz:masa") (at 273.7468 22.8563 0) (unit 1)
     (in_bom yes) (on_board yes) (dnp no) (fields_autoplaced)
@@
     )
   )
+  (symbol (lib_id "sp3jdz:masa") (at 27.305 59.055 0) (unit 1)
+    (in_bom yes) (on_board yes) (dnp no) (fields_autoplaced)
+    (property "Reference" "#PWR07" (at 27.305 65.405 0)
+      (effects (font (size 1.27 1.27)) hide)
+    )
+    (property "Value" "masa" (at 27.305 61.595 0)
+      (effects (font (size 0.9906 0.9906)) hide)
+    )
+    (property "Footprint" "" (at 27.305 59.055 0)
+      (effects (font (size 1.524 1.524)))
+    )
+    (property "Datasheet" "" (at 27.305 59.055 0)
+      (effects (font (size 1.524 1.524)))
+    )
+    (pin "1")
+    (instances
+      (project "password_manager"
+        (path "/c60f1c42-9579-4917-bb90-9d2f0e5f1bce"
+          (reference "#PWR07") (unit 1)
+        )
+      )
+    )
+  )
   (symbol (lib_id "Device:C_Small") (at 99.695 60.325 0) (unit 1)
     (in_bom yes) (on_board yes) (dnp no) (fields_autoplaced)
@@
         )
       )
+    )
+  )
+  (symbol (lib_id "sp3jdz:masa") (at 19.685 59.055 0) (unit 1)
+    (in_bom yes) (on_board yes) (dnp no) (fields_autoplaced)
+    (property "Reference" "#PWR08" (at 19.685 65.405 0)
+      (effects (font (size 1.27 1.27)) hide)
+    )
+    (property "Value" "masa" (at 19.685 61.595 0)
+      (effects (font (size 0.9906 0.9906)) hide)
+    )
+    (property "Footprint" "" (at 19.685 59.055 0)
+      (effects (font (size 1.524 1.524)))
+    )
+    (property "Datasheet" "" (at 19.685 59.055 0)
+      (effects (font (size 1.524 1.524)))
+    )
+    (pin "1")
+    (instances
+      (project "password_manager"
+        (path "/c60f1c42-9579-4917-bb90-9d2f0e5f1bce"
+          (reference "#PWR08") (unit 1)
+        )
+      )
+    )
+  )
+  (symbol (lib_id "Connector:USB_C_Receptacle_USB2.0") (at 64.135 36.195 0) (unit 1)
+    (in_bom yes) (on_board yes) (dnp no) (fields_autoplaced)
+    (property "Reference" "J4" (at 64.135 13.97 0)
+      (effects (font (size 1.27 1.27)))
+    )
+    (property "Value" "USB_C_Receptacle_USB2.0" (at 64.135 16.51 0)
+      (effects (font (size 1.27 1.27)))
+    )
+    (property "Footprint" "Connector_USB:USB_C_Receptacle_GCT_USB4105-xx-A_16P_TopMnt_Horizontal" (at 67.945 36.195 0)
+      (effects (font (size 1.27 1.27)) hide)
+    )
+    (property "Datasheet" "https://www.usb.org/sites/default/files/documents/usb_type-c.zip" (at 67.945 36.195 0)
+      (effects (font (size 1.27 1.27)) hide)
+    )
+    (pin "B4")
+    (pin "A5")
+    (pin "A1")
+    (pin "B6")
+    (pin "B8")
+    (pin "S1")
+    (pin "A12")
+    (pin "B7")
+    (pin "B1")
+    (pin "B5")
+    (pin "B12")
+    (pin "A7")
+    (pin "A4")
+    (pin "A9")
+    (pin "B9")
+    (pin "A6")
+    (pin "A8")
+    (instances
+      (project "password_manager"
+        (path "/c60f1c42-9579-4917-bb90-9d2f0e5f1bce"
+          (reference "J4") (unit 1)
+        )
+      )

Commit message: kolejne elementy
Parts:
- added CON1: ISP-10, foots:IDC-10_angled, symbol sp3jdz:ISP-10
- added D1, D2, D3, D4: LED_Small, Diode_SMD:D_0805_2012Metric_Pad1.15x1.40mm_HandSolder, symbol Device:LED_Small
- added J10, J9: Conn_01x22_Pin, Connector_PinHeader_2.54mm:PinHeader_1x22_P2.54mm_Vertical, symbol Connector:Conn_01x22_Pin
- added J11, J12, J13, J14: masa_pomiarowa, foots:masa_pomiarowa, symbol Connector:Conn_01x01_Pin
- added J15: LEDS, foots:4_PIN, symbol Connector:Conn_01x04_Pin
- added J16, J17, J18, J19, J20, J21: test_pin, foots:3_PIN, symbol Connector:Conn_01x03_Pin
- added J6: RJ45_Shielded, password_manager_foots:RJ45_6339160-1_TE_Connectivity, symbol Connector:RJ45_Shielded
- added J7, J8: Conn_01x22_Pin, Connector_PinHeader_2.54mm:PinHeader_1x22_P2.54mm_Horizontal, symbol Connector:Conn_01x22_Pin
- added R1: R_Small, Resistor_SMD:R_0805_2012Metric_Pad1.20x1.40mm_HandSolder, symbol Device:R_Small
- added R2: 10K, Resistor_SMD:R_0805_2012Metric_Pad1.20x1.40mm_HandSolder, symbol Device:R_Small
- added SW1: SW_Push, Button_Switch_SMD:SW_Push_1P1T_NO_6x6mm_H9.5mm, symbol Switch:SW_Push
Connections:
- net GND: now also J11.1 (Pin_1), J12.1 (Pin_1), J13.1 (Pin_1), J14.1 (Pin_1), SW1.1
- net at U1.14 (NRST): now also R2.2, SW1.2
- new net: D1.2 (A), R1.2
- new net: D1.1 (K), J15.1 (Pin_1)
- new net +3,3V: R1.1, R2.1
